Commit message: Removed gripper

File: ridgeback/ridgeback_description/urdf/accessories.urdf.xacro (robot description, xacro)
@@ -11,6 +11,5 @@
   <xacro:include filename="$(find ridgeback_description)/urdf/accessories/sick_lms1xx_mount.urdf.xacro" />
   <xacro:include filename="$(find ridgeback_description)/urdf/accessories/hokuyo_ust-10lx_mount.urdf.xacro" />
-  <xacro:include filename="$(find ur_description)/urdf/ur10.urdf.xacro" />
-  <xacro:include filename="$(find robotiq_s_model_visualization)/cfg/s-model_articulated_macro.xacro" />
+  <xacro:include filename="$(find ur_description)/urdf/ur5.urdf.xacro" />
   <!-- If enabled, generate the front HOKUYO UST-10LX LASER payload. -->
   <xacro:if value="$(optenv RIDGEBACK_FRONT_HOKUYO_LASER 0)">
@@ -55,17 +54,10 @@
   </joint>
 <!-- Spawn arm -->
-  <xacro:ur10_robot prefix="ur10_arm_" joint_limited="true"/>
+  <xacro:ur5_robot prefix="ur5_arm_" joint_limited="true"/>
   <!-- Join arm -->
-  <joint name="ur10_arm_base" type="fixed">
+  <joint name="ur5_arm_base" type="fixed">
 	<parent link="arch_link" />
-	<child link="ur10_arm_base_link" />
+	<child link="ur5_arm_base_link" />
 	<origin xyz="0.01 -0.27 0.375" rpy="0.0 0.0 3.1416" />
-  </joint>
-  <!-- Spawn and Join Gripper -->
-  <xacro:s-model_articulated prefix="" />
-  <joint name="gripper_base" type="fixed">
-	<parent link="ur10_arm_ee_link" />
-	<child link="palm" />
-	<origin xyz="0.11 0.0 0.0" rpy="0.0 -0.786 -1.57" />
   </joint>
   <!-- Sensor Mount and other custom parts -->
@@ -85,5 +77,5 @@
   <joint name="FT300_joint" type="fixed">
 	  <origin xyz="0.03 0 0" rpy="0 1.57 0" />
-	  <parent link="ur10_arm_ee_link" />
+	  <parent link="ur5_arm_ee_link" />
 	  <child link="FT300_link" />
   </joint>

Commit message: Changed to EPFL01 Layout from old mech arch

File: ridgeback/ridgeback_description/urdf/accessories.urdf.xacro (robot description, xacro)
@@ -39,10 +39,10 @@
 		<visual>
 			<geometry>
-				<mesh filename="package://ridgeback_description/meshes/tor11_mech.dae" />
+				<mesh filename="package://ridgeback_description/meshes/epfl_arch.dae" />
 			</geometry>
 		</visual>
 		<collision>
 			<geometry>
-				<mesh filename="package://ridgeback_description/meshes/tor11_mech.dae" />
+				<mesh filename="package://ridgeback_description/meshes/epfl_arch.dae" />
 			</geometry>
 		</collision>

Commit message: Added extra install to readme, tuning positions of accessories

File: ridgeback/ridgeback_description/urdf/accessories.urdf.xacro (robot description, xacro)
@@ -49,5 +49,5 @@
    </link>
   <joint name="arch_joint" type="fixed">
-	  <origin xyz="0 0 0.278" rpy="0 0 1.5" />
+	  <origin xyz="-0.38 0 0.278" rpy="0 0 1.5" />
 	  <parent link="top_link" />
 	  <child link="arch_link" />
@@ -57,7 +57,7 @@
   <!-- Join arm -->
   <joint name="ur5_arm_base" type="fixed">
-	<parent link="arch_link" />
+	<parent link="mid_mount" />
 	<child link="ur5_arm_base_link" />
-	<origin xyz="0.01 -0.27 0.375" rpy="0.0 0.0 3.1416" />
+	<origin xyz="0.22 0.0 0.0" rpy="0.0 0.0 -1.5708" />
   </joint>
   <!-- Sensor Mount and other custom parts -->
@@ -65,5 +65,5 @@
 		<visual>
 			<geometry>
-				<cylinder length="0.06" radius="0.035"/>
+				<cylinder length="0.04" radius="0.035"/>
 			</geometry>
 			<material name="black"/>
@@ -71,10 +71,10 @@
 		<collision>
 			<geometry>
-				<cylinder length="0.0475" radius="0.035"/>
+				<cylinder length="0.04" radius="0.035"/>
 			</geometry>
 		</collision>
    </link>
   <joint name="FT300_joint" type="fixed">
-	  <origin xyz="0.03 0 0" rpy="0 1.57 0" />
+	  <origin xyz="0.02 0 0" rpy="0 1.57 0" />
 	  <parent link="ur5_arm_ee_link" />
 	  <child link="FT300_link" />
